Commit message: [FIX indent]

File: sobit_pro_description/urdf/base/base.urdf.xacro (robot description, xacro)
@@ -1,12 +1,13 @@
 <?xml version="1.0" encoding="UTF-8" ?>
-<robot name="base" xmlns:xacro="http://ros.org/wiki/xacro" >
-    <xacro:macro name="base" >
-        <link name="base_footprint" />
-        <joint name="base_joint" type="fixed" >
-            <parent link="base_footprint" />
-            <child link="base_link" />
-            <origin xyz="0 0 0.177" rpy="0.0 0.0 0.0" />
-        </joint>
-        <link name="base_link" />
-    </xacro:macro>
+<robot name="sobit_pro"
+       xmlns:xacro="http://ros.org/wiki/xacro" >
+  <xacro:macro name="base" >
+    <link name="base_footprint" />
+    <joint name="base_joint" type="fixed" >
+      <parent link="base_footprint" />
+      <child link="base_link" />
+      <origin xyz="0 0 0.177" rpy="0.0 0.0 0.0" />
+    </joint>
+    <link name="base_link" />
+  </xacro:macro>
 </robot>
