Commit message: [FIX] robot name

File: sobit_pro_description/urdf/body/cover.urdf.xacro (robot description, xacro)
@@ -1,4 +1,5 @@
 <?xml version="1.0" encoding="UTF-8" ?>
-<robot name="cover" xmlns:xacro="http://ros.org/wiki/xacro" >
+<robot name="sobit_pro"
+       xmlns:xacro="http://ros.org/wiki/xacro" >
   <xacro:macro name="cover" params="prefix parent" >
     <joint name="${prefix}_joint" type="fixed" >

File: sobit_pro_description/urdf/body/plate.urdf.xacro (robot description, xacro)
@@ -1,5 +1,6 @@
 <?xml version="1.0" encoding="UTF-8" ?>
-<robot name="plate" xmlns:xacro="http://ros.org/wiki/xacro">
-    <xacro:macro name="plate" params="prefix parent">
+<robot name="sobit_pro"
+       xmlns:xacro="http://ros.org/wiki/xacro" >
+  <xacro:macro name="plate" params="prefix parent">
     <joint name="${prefix}_bottom_joint" type="fixed">
       <origin xyz="0.0 0.0 0.0" rpy="0.0 0.0 0.0" />
@@ -98,4 +99,4 @@
       </inertial>
     </link>
-    </xacro:macro>
+  </xacro:macro>
 </robot>
