Commit message: [FIX] reduce virtual link

File: sobit_pro_description/urdf/hand/hand.urdf.xacro (robot description, xacro)
@@ -1,4 +1,5 @@
 <?xml version="1.0" encoding="UTF-8" ?>
-<robot name="hand" xmlns:xacro="http://ros.org/wiki/xacro">
+<robot name="sobit_pro"
+       xmlns:xacro="http://ros.org/wiki/xacro" >
   <xacro:include filename="$(find sobit_pro_description)/urdf/hand/hand.transmission.xacro" />
   <xacro:macro name="hand" params="prefix_hand prefix_finger parent">
@@ -35,5 +36,5 @@
       </inertial>
     </link>
-    <joint name="${prefix_hand}_joint" type="revolute">
+    <!-- <joint name="${prefix_hand}_joint" type="revolute">
       <parent link="${prefix_hand}_base_link" />
       <child link="${prefix_hand}_link" />
@@ -42,5 +43,5 @@
       <limit lower="${-M_PI/2.0}" upper="0" effort="1" velocity="1" />
     </joint>
-    <link name="${prefix_hand}_link" />
+    <link name="${prefix_hand}_link" /> -->
     <joint name="${prefix_hand}_inner_l_joint" type="revolute">
       <parent link="${prefix_hand}_base_link" />
@@ -78,13 +79,13 @@
       </inertial>
     </link>
-    <joint name="${prefix_hand}_inner_r_joint" type="revolute">
-      <parent link="${prefix_hand}_base_link" />
-      <child link="${prefix_hand}_inner_r_link" />
+    <joint name="${prefix_hand}_joint" type="revolute">
+      <parent link="${prefix_hand}_base_link" />
+      <child link="${prefix_hand}_link" />
       <origin xyz="0.0631932 -0.0151495 0.0372231" rpy="0.0 0.0 0.0" />
       <axis xyz="0.0 0.0 1.0" />
-      <mimic joint="${prefix_hand}_joint" multiplier="1.0" offset="0" />
-      <limit lower="${-M_PI/2.0}" upper="0" effort="1" velocity="1" />
-    </joint>
-    <link name="${prefix_hand}_inner_r_link">
+      <!-- <mimic joint="${prefix_hand}_joint" multiplier="1.0" offset="0" /> -->
+      <limit lower="${-M_PI/2.0}" upper="0" effort="1" velocity="1" />
+    </joint>
+    <link name="${prefix_hand}_link">
       <visual>
         <origin xyz="0.0 0.0 0.0" rpy="0.0 0.0 ${M_PI/2.0}" />
@@ -223,5 +224,5 @@
     </link>
     <joint name="${prefix_hand}_${prefix_finger}_r_joint" type="revolute">
-      <parent link="${prefix_hand}_inner_r_link" />
+      <parent link="${prefix_hand}_link" />
       <child link="${prefix_hand}_${prefix_finger}_r_link" />
       <origin xyz="0.114316 0.0 -0.027729" rpy="0.0 0.0 0.0" />
