Commit message: [UPD] clean up

File: sobit_pro_description/urdf/back/back.urdf.xacro (robot description, xacro)
@@ -18,8 +18,6 @@
       <collision>
         <origin xyz="0.0 0.0 ${0.517/2}" rpy="0.0 0.0 0.0" />
-        <!-- <origin xyz="0.0 0.0 0.0" rpy="0.0 0.0 ${M_PI}" /> -->
         <geometry>
           <box size="0.02 0.02 0.517"/>
-          <!-- <mesh filename="package://sobit_pro_description/meshes/back/back_base.stl" scale="0.001 0.001 0.001" /> -->
         </geometry>
       </collision>
@@ -30,7 +28,4 @@
                  iyy="${1/12*0.5*(0.02**2+0.517**2)}" iyz="0.0"
                  izz="${1/12*0.5*(0.02**2+0.02**2)}" />
-        <!-- <inertia ixx="1.0" ixy="0.0" ixz="0.0"
-                 iyy="1.0" iyz="0.0"
-                 izz="1.0" /> -->
       </inertial>
     </link>

File: sobit_pro_description/urdf/body/cover.urdf.xacro (robot description, xacro)
@@ -18,8 +18,6 @@
       <collision>
         <origin xyz="-${0.02893+0.3/2} 0.0 ${0.034-0.489/2}" rpy="0.0 0.0 0.0" />
-        <!-- <origin xyz="0.0 0.0 0.0" rpy="${M_PI/2} 0.0 ${M_PI/2}" /> -->
         <geometry>
           <box size="${(0.02893+0.3/2)*2} 0.3965 0.489"/>
-          <!-- <mesh filename="package://sobit_pro_description/meshes/body/cover.stl" scale="0.001 0.001 0.001" /> -->
         </geometry>
       </collision>
@@ -30,7 +28,4 @@
                  iyy="${1/12*0.732*(0.3965**2+0.489**2)}"               iyz="0.0"
                  izz="${1/12*0.732*(((0.02893+0.3/2)*2)**2+0.3965**2)}" />
-        <!-- <inertia ixx="0.0001" ixy="0.0" ixz="0.0"
-                 iyy="0.0001" iyz="0.0"
-                 izz="0.0001" /> -->
       </inertial>
     </link>

File: sobit_pro_description/urdf/body/plate.urdf.xacro (robot description, xacro)
@@ -18,8 +18,6 @@
       <collision>
         <origin xyz="0.0 0.0 -${0.009/2}" rpy="0.0 0.0 0.0" />
-        <!-- <origin xyz="0.0 0.0 0.0" rpy="0.0 0.0 0.0" /> -->
         <geometry>
           <box size="0.3 0.3 0.009" />
-          <!-- <mesh filename="package://sobit_pro_description/meshes/body/plate_bottom.stl" scale="0.001 0.001 0.001" /> -->
         </geometry>
       </collision>
@@ -30,7 +28,4 @@
                  iyy="${1/12*0.08*(0.3**2+0.009**2)}" iyz="0.0"
                  izz="${1/12*0.08*(0.3**2+0.3**2)}" />
-        <!-- <inertia ixx="1.0" ixy="0.0" ixz="0.0"
-                 iyy="1.0" iyz="0.0"
-                 izz="1.0" /> -->
       </inertial>
     </link>
@@ -50,8 +45,6 @@
       <collision>
         <origin xyz="0.0 0.0 -${0.009/2}" rpy="0.0 0.0 0.0" />
-        <!-- <origin xyz="0.0 0.0 0.0" rpy="0.0 0.0 0.0" /> -->
         <geometry>
           <box size="0.3 0.3 0.009" />
-          <!-- <mesh filename="package://sobit_pro_description/meshes/body/plate_middle.stl" scale="0.001 0.001 0.001" /> -->
         </geometry>
       </collision>
@@ -62,7 +55,4 @@
                  iyy="${1/12*0.08*(0.3**2+0.009**2)}" iyz="0.0"
                  izz="${1/12*0.08*(0.3**2+0.3**2)}" />
-        <!-- <inertia ixx="1.0" ixy="0.0" ixz="0.0"
-                 iyy="1.0" iyz="0.0"
-                 izz="1.0" /> -->
       </inertial>
     </link>
@@ -82,8 +72,6 @@
       <collision>
         <origin xyz="0.0 0.0 -${0.009/2}" rpy="0.0 0.0 0.0" />
-        <!-- <origin xyz="0.0 0.0 0.0" rpy="0.0 0.0 ${M_PI/2}" /> -->
         <geometry>
           <box size="0.3 0.3 0.009" />
-          <!-- <mesh filename="package://sobit_pro_description/meshes/body/plate_top.stl" scale="0.001 0.001 0.001" /> -->
         </geometry>
       </collision>
@@ -94,7 +82,4 @@
                  iyy="${1/12*0.08*(0.3**2+0.009**2)}" iyz="0.0"
                  izz="${1/12*0.08*(0.3**2+0.3**2)}" />
-        <!-- <inertia ixx="1.0" ixy="0.0" ixz="0.0"
-                 iyy="1.0" iyz="0.0"
-                 izz="1.0" /> -->
       </inertial>
     </link>

File: sobit_pro_description/urdf/sensor/lidar.urdf.xacro (robot description, xacro)
@@ -18,8 +18,6 @@
       <collision>
         <origin xyz="${0.092/2} 0.0 -${0.007/2}" rpy="0.0 0.0 0.0" />
-        <!-- <origin xyz="0.0 0.0 0.0" rpy="${M_PI/2} 0.0 ${M_PI}" /> -->
         <geometry>
           <box size="0.092 0.184 0.007"/>
-          <!-- <mesh filename="package://sobit_pro_description/meshes/sensor/lidar_base.stl" scale="0.001 0.001 0.001" /> -->
         </geometry>
       </collision>
@@ -30,7 +28,4 @@
                  iyy="${1/12*0.08*(0.184**2+0.007**2)}" iyz="0.0"
                  izz="${1/12*0.08*(0.092**2+0.184**2)}" />
-        <!-- <inertia ixx="1.0" ixy="0.0" ixz="0.0"
-                 iyy="1.0" iyz="0.0"
-                 izz="1.0" /> -->
       </inertial>
     </link>

File: sobit_pro_description/urdf/sensor/mic.urdf.xacro (robot description, xacro)
@@ -18,8 +18,6 @@
       <collision>
         <origin xyz="0.0 ${(0.02-0.1146-0.0146)/2} -${0.02/2}" rpy="0.0 0.0 0.0" />
-        <!-- <origin xyz="0.0 0.0 0.0" rpy="${M_PI/2} 0.0 ${M_PI}" /> -->
         <geometry>
           <box size="0.0292 ${0.1146+0.0146} 0.03"/>
-          <!-- <mesh filename="package://sobit_pro_description/meshes/sensor/mic_base.stl" scale="0.001 0.001 0.001" /> -->
         </geometry>
         <material name="black" />
@@ -32,7 +30,4 @@
                  iyy="${1/12*0.15*((0.1146+0.0146)**2+0.03**2)}"   iyz="0.0"
                  izz="${1/12*0.15*(0.0292**2+(0.1146+0.0146)**2)}" />
-        <!-- <inertia ixx="1.0" ixy="0.0" ixz="0.0"
-                 iyy="1.0" iyz="0.0"
-                 izz="1.0" /> -->
       </inertial>
     </link>
@@ -52,8 +47,6 @@
       <collision>
         <origin xyz="${0.0+0.04911} -${0.0112/2} ${0.035+0.0266}" rpy="0.0 ${M_PI/2-25*M_PI/180} 0.0" />
-        <!-- <origin xyz="0.0 0.0 0.0" rpy="${M_PI/2} 0.0 ${M_PI}" /> -->
         <geometry>
           <cylinder radius="${0.022/2}" length="0.281"/>
-          <!-- <mesh filename="package://sobit_pro_description/meshes/sensor/mic.stl" scale="0.001 0.001 0.001" /> -->
         </geometry>
         <material name="black" />
