Commit message: [FIX] parallel joints are ommited

File: sobit_pro_sim_description/urdf/arm/arm.transmission.xacro (robot description, xacro)
@@ -4,7 +4,7 @@
   <xacro:macro name="arm_transmission" params="prefix">
     <xacro:position_joint_transmission joint="${prefix}_shoulder_1_tilt_joint"    reduction="1" />
-    <xacro:position_joint_transmission joint="${prefix}_shoulder_2_tilt_joint"    reduction="1" />
+    <!-- <xacro:position_joint_transmission joint="${prefix}_shoulder_2_tilt_joint"    reduction="1" /> -->
     <xacro:position_joint_transmission joint="${prefix}_elbow_upper_1_tilt_joint" reduction="1" />
-    <xacro:position_joint_transmission joint="${prefix}_elbow_upper_2_tilt_joint" reduction="1" />
+    <!-- <xacro:position_joint_transmission joint="${prefix}_elbow_upper_2_tilt_joint" reduction="1" /> -->
     <xacro:position_joint_transmission joint="${prefix}_elbow_lower_tilt_joint"   reduction="1" />
     <xacro:position_joint_transmission joint="${prefix}_elbow_lower_pan_joint"    reduction="1" />

File: sobit_pro_sim_description/urdf/arm/arm.urdf.xacro (robot description, xacro)
@@ -2,5 +2,5 @@
 <robot name="sobit_pro"
        xmlns:xacro="http://ros.org/wiki/xacro" >
-  <xacro:include filename="$(find sobit_pro_description)/urdf/arm/arm.transmission.xacro" />
+  <xacro:include filename="$(find sobit_pro_sim_description)/urdf/arm/arm.transmission.xacro" />
   <xacro:macro name="arm" params="prefix parent" >
     <joint name="${prefix}_base_joint" type="fixed" >
@@ -61,5 +61,5 @@
       </inertial>
     </link>
-    <joint name="${prefix}_shoulder_2_tilt_joint" type="revolute" >
+    <!-- <joint name="${prefix}_shoulder_2_tilt_joint" type="revolute" >
       <parent link="${prefix}_base_link" />
       <child link="${prefix}_shoulder_2_tilt_link" />
@@ -68,7 +68,7 @@
       <mimic joint="${prefix}_shoulder_1_tilt_joint" multiplier="1" offset="0" />
       <limit lower="${-M_PI/2}" upper="${M_PI/2}" effort="25" velocity="11.031179004" />
-      <!-- <dynamics damping="0.2" friction="0" /> -->
-    </joint>
-    <link name="${prefix}_shoulder_2_tilt_link" />
+      <dynamics damping="0.2" friction="0" />
+    </joint> -->
+    <!-- <link name="${prefix}_shoulder_2_tilt_link" /> -->
     <joint name="${prefix}_elbow_upper_1_tilt_joint" type="revolute" >
       <parent link="${prefix}_shoulder_1_tilt_link" />
@@ -101,5 +101,5 @@
       </inertial>
     </link>
-    <joint name="${prefix}_elbow_upper_2_tilt_joint" type="revolute" >
+    <!-- <joint name="${prefix}_elbow_upper_2_tilt_joint" type="revolute" >
       <parent link="${prefix}_shoulder_1_tilt_link" />
       <child link="${prefix}_elbow_upper_2_tilt_link" />
@@ -108,7 +108,7 @@
       <mimic joint="${prefix}_elbow_upper_1_tilt_joint" multiplier="1" offset="0" />
       <limit lower="${-M_PI/2}" upper="${M_PI/2}" effort="25" velocity="9.59233" />
-      <!-- <dynamics damping="0.2" friction="0" /> -->
-    </joint>
-    <link name="${prefix}_elbow_upper_2_tilt_link" />
+      <dynamics damping="0.2" friction="0" />
+    </joint> -->
+    <!-- <link name="${prefix}_elbow_upper_2_tilt_link" /> -->
     <joint name="${prefix}_elbow_lower_tilt_joint" type="revolute" >
       <parent link="${prefix}_elbow_upper_1_tilt_link" />
