Commit message: [UPD] fix effort values

File: sobit_pro_sim_description/urdf/arm/arm.urdf.xacro (robot description, xacro)
@@ -36,5 +36,5 @@
       <origin xyz="0.1560 0.0 0.0215" rpy="0.0 0.0 0.0 " />
       <axis xyz="0.0 -1.0 0.0 " />
-      <limit lower="${-M_PI/2}" upper="${M_PI/2}" effort="25" velocity="11.031179004" />
+      <limit lower="${-M_PI/2}" upper="${M_PI/2}" effort="${10.6*2}" velocity="11.031179004" />
       <!-- <dynamics damping="0.2" friction="0" /> -->
     </joint>
@@ -67,5 +67,5 @@
       <axis xyz="0.0 1.0 0.0 " />
       <mimic joint="${prefix}_shoulder_1_tilt_joint" multiplier="1" offset="0" />
-      <limit lower="${-M_PI/2}" upper="${M_PI/2}" effort="25" velocity="11.031179004" />
+      <limit lower="${-M_PI/2}" upper="${M_PI/2}" effort="${10.6*2}" velocity="11.031179004" />
       <dynamics damping="0.2" friction="0" />
     </joint> -->
@@ -76,5 +76,5 @@
       <origin xyz="0.1500 0.0 0.0" rpy="0.0 0.0 0.0" />
       <axis xyz="0.0 -1.0 0.0 " />
-      <limit lower="${-M_PI/2}" upper="${M_PI/2}" effort="25" velocity="9.59233" />
+      <limit lower="${-M_PI/2}" upper="${M_PI/2}" effort="${4.1*2}" velocity="9.59233" />
       <!-- <dynamics damping="0.2" friction="0" /> -->
     </joint>
@@ -107,5 +107,5 @@
       <axis xyz="0.0 1.0 0.0 " />
       <mimic joint="${prefix}_elbow_upper_1_tilt_joint" multiplier="1" offset="0" />
-      <limit lower="${-M_PI/2}" upper="${M_PI/2}" effort="25" velocity="9.59233" />
+      <limit lower="${-M_PI/2}" upper="${M_PI/2}" effort="${4.1*2}" velocity="9.59233" />
       <dynamics damping="0.2" friction="0" />
     </joint> -->
@@ -116,5 +116,5 @@
       <origin xyz="0.1500 0.0 0.0" rpy="0.0 0.0 0.0" />
       <axis xyz="0.0 -1.0 0.0 " />
-      <limit lower="${-M_PI/2}" upper="${M_PI/2}" effort="25" velocity="4.796165" />
+      <limit lower="${-M_PI/2}" upper="${M_PI/2}" effort="4.1" velocity="4.796165" />
       <!-- <dynamics damping="0.2" friction="0" /> -->
     </joint>
@@ -146,5 +146,5 @@
       <origin xyz="0.028 0.0 0.0" rpy="0.0 0.0 0.0" />
       <axis xyz="1.0 0.0 0.0 " />
-      <limit lower="${-M_PI/2}" upper="${M_PI/2}" effort="25" velocity="4.796165" />
+      <limit lower="${-M_PI/2}" upper="${M_PI/2}" effort="4.1" velocity="4.796165" />
       <!-- <dynamics damping="0.2" friction="0" /> -->
     </joint>
@@ -176,5 +176,5 @@
       <origin xyz="0.122009 0.0 0.0" rpy="0.0 0.0 0.0" />
       <axis xyz="0.0 -1.0 0.0" />
-      <limit lower="${-M_PI/2}" upper="${M_PI/2}" effort="25" velocity="4.796165" />
+      <limit lower="${-M_PI/2}" upper="${M_PI/2}" effort="4.1" velocity="4.796165" />
       <!-- <dynamics damping="0.2" friction="0" /> -->
     </joint>
