Commit message: [UPD] add mimic joints

File: sobit_pro_sim_description/urdf/gazebo.urdf.xacro (robot description, xacro)
@@ -2,5 +2,24 @@
 <robot name="sobit_pro"
        xmlns:xacro="http://www.ros.org/wiki.xacro">
+  <xacro:macro name="mimic_joint" params="name_prefix parent_joint mimic_joint has_pid:=false multiplier:=1.0 offset:=0 sensitiveness:=0.0 max_effort:=1.0 robot_namespace:=''">
+    <gazebo>
+      <plugin name="${name_prefix}_mimic_joint_plugin" filename="libroboticsgroup_upatras_gazebo_mimic_joint_plugin.so">
+        <joint>${parent_joint}</joint>
+        <mimicJoint>${mimic_joint}</mimicJoint>
+        <xacro:if value="${has_pid}">                     <!-- if set to true, PID parameters from "/gazebo_ros_control/pid_gains/${mimic_joint}" are loaded -->
+          <hasPID />
+        </xacro:if>
+        <multiplier>${multiplier}</multiplier>
+        <offset>${offset}</offset>
+        <sensitiveness>${sensitiveness}</sensitiveness>   <!-- if absolute difference between setpoint and process value is below this threshold, do nothing; 0.0 = disable [rad] -->
+        <maxEffort>${max_effort}</maxEffort>              <!-- only taken into account if has_pid:=true [Nm] -->
+        <xacro:unless value="${robot_namespace == ''}">
+          <robotNamespace>${robot_namespace}</robotNamespace>
+        </xacro:unless>
+      </plugin>
+    </gazebo>
+  </xacro:macro>
   <xacro:macro name="gazebo">
+    <!-- Gazebo -->
     <gazebo>
       <plugin name="gazebo_ros_control" filename="libgazebo_ros_control.so">
@@ -10,4 +29,50 @@
       </plugin>
     </gazebo>
+    <!-- Mimic Joints -->
+    <xacro:mimic_joint
+      name_prefix="hand_inner_l_joint"
+      parent_joint="hand_joint"
+      mimic_joint="hand_inner_l_joint"
+      has_pid="false"
+      multiplier="-1.0"
+      max_effort="10.0"
+      robot_namespace="$(arg robot_namespace)"
+    />
+    <xacro:mimic_joint
+      name_prefix="hand_outer_l_joint"
+      parent_joint="hand_joint"
+      mimic_joint="hand_outer_l_joint"
+      has_pid="false"
+      multiplier="-1.0"
+      max_effort="10.0"
+      robot_namespace="$(arg robot_namespace)"
+    />
+    <xacro:mimic_joint
+      name_prefix="hand_outer_r_joint"
+      parent_joint="hand_joint"
+      mimic_joint="hand_outer_r_joint"
+      has_pid="false"
+      multiplier="1.0"
+      max_effort="10.0"
+      robot_namespace="$(arg robot_namespace)"
+    />
+    <xacro:mimic_joint
+      name_prefix="hand_finger_l_joint"
+      parent_joint="hand_joint"
+      mimic_joint="hand_finger_l_joint"
+      has_pid="false"
+      multiplier="1.0"
+      max_effort="10.0"
+      robot_namespace="$(arg robot_namespace)"
+    />
+    <xacro:mimic_joint
+      name_prefix="hand_finger_r_joint"
+      parent_joint="hand_joint"
+      mimic_joint="hand_finger_r_joint"
+      has_pid="false"
+      multiplier="-1.0"
+      max_effort="10.0"
+      robot_namespace="$(arg robot_namespace)"
+    />
     <!-- Arm -->
     <gazebo reference="arm_base_link">
