Commit message: [UPD] unable dynamics and fix style

File: sobit_pro_description/urdf/arm/arm.urdf.xacro (robot description, xacro)
@@ -1,4 +1,5 @@
 <?xml version="1.0" encoding="UTF-8" ?>
-<robot name="arm" xmlns:xacro="http://ros.org/wiki/xacro" >
+<robot name="sobit_pro"
+       xmlns:xacro="http://ros.org/wiki/xacro" >
   <xacro:include filename="$(find sobit_pro_description)/urdf/arm/arm.transmission.xacro" />
   <xacro:macro name="arm" params="prefix parent" >
@@ -40,5 +41,5 @@
       <origin xyz="0.1560 0.0 0.0215" rpy="0.0 0.0 0.0 " />
       <axis xyz="0.0 -1.0 0.0 " />
-      <limit lower="${-M_PI / 2}" upper="${M_PI/2}" effort="10" velocity="10" />
+      <limit lower="${-M_PI/2}" upper="${M_PI/2}" effort="10" velocity="10" />
       <!-- <dynamics damping="0.2" friction="0" /> -->
     </joint>
@@ -76,6 +77,6 @@
       <axis xyz="0.0 1.0 0.0 " />
       <mimic joint="${prefix}_shoulder_1_tilt_joint" multiplier="1" offset="0" />
-      <limit lower="${-M_PI / 2}" upper="${M_PI/2}" effort="10" velocity="10" />
-      <dynamics damping="0.2" friction="0" />
+      <limit lower="${-M_PI/2}" upper="${M_PI/2}" effort="10" velocity="10" />
+      <!-- <dynamics damping="0.2" friction="0" /> -->
     </joint>
     <link name="${prefix}_shoulder_2_tilt_link" />
@@ -85,5 +86,5 @@
       <origin xyz="0.1500 0.0 0.0" rpy="0.0 0.0 0.0" />
       <axis xyz="0.0 -1.0 0.0 " />
-      <limit lower="${-M_PI / 2}" upper="${M_PI/2}" effort="10" velocity="10" />
+      <limit lower="${-M_PI/2}" upper="${M_PI/2}" effort="10" velocity="10" />
       <!-- <dynamics damping="0.2" friction="0" /> -->
     </joint>
@@ -121,6 +122,6 @@
       <axis xyz="0.0 1.0 0.0 " />
       <mimic joint="${prefix}_elbow_upper_1_tilt_joint" multiplier="1" offset="0" />
-      <limit lower="${-M_PI / 2}" upper="${M_PI/2}" effort="10" velocity="10" />
-      <dynamics damping="0.2" friction="0" />
+      <limit lower="${-M_PI/2}" upper="${M_PI/2}" effort="10" velocity="10" />
+      <!-- <dynamics damping="0.2" friction="0" /> -->
     </joint>
     <link name="${prefix}_elbow_upper_2_tilt_link" />
@@ -130,5 +131,5 @@
       <origin xyz="0.1500 0.0 0.0" rpy="0.0 0.0 0.0" />
       <axis xyz="0.0 -1.0 0.0 " />
-      <limit lower="${-M_PI / 2}" upper="${M_PI/2}" effort="10" velocity="10" />
+      <limit lower="${-M_PI/2}" upper="${M_PI/2}" effort="10" velocity="10" />
       <!-- <dynamics damping="0.2" friction="0" /> -->
     </joint>
@@ -165,5 +166,5 @@
       <origin xyz="0.028 0.0 0.0" rpy="0.0 0.0 0.0" />
       <axis xyz="1.0 0.0 0.0 " />
-      <limit lower="${-M_PI / 2}" upper="${M_PI/2}" effort="10" velocity="10" />
+      <limit lower="${-M_PI/2}" upper="${M_PI/2}" effort="10" velocity="10" />
       <!-- <dynamics damping="0.2" friction="0" /> -->
     </joint>
@@ -201,5 +202,5 @@
       <origin xyz="0.122009 0.0 0.0" rpy="0.0 0.0 0.0" />
       <axis xyz="0.0 -1.0 0.0" />
-      <limit lower="${-M_PI / 2}" upper="${M_PI/2}" effort="10" velocity="10" />
+      <limit lower="${-M_PI/2}" upper="${M_PI/2}" effort="10" velocity="10" />
       <!-- <dynamics damping="0.2" friction="0" /> -->
     </joint>
