Commit message: [UPD] velocities and effort limits are updated based on real robot

File: sobit_pro_description/urdf/arm/arm.urdf.xacro (robot description, xacro)
@@ -19,8 +19,6 @@
       <collision>
         <origin xyz="${0.140/2} 0.0 ${0.043/2}" rpy="0.0 0.0 0.0" />
-        <!-- <origin xyz="0.0 0.0 0.0" rpy="${M_PI/2} 0.0 0.0" /> -->
         <geometry>
           <box size="0.140 0.156 0.043" />
-          <!-- <mesh filename="package://sobit_pro_description/meshes/arm/arm_base.stl" scale="0.001 0.001 0.001" /> -->
         </geometry>
       </collision>
@@ -31,7 +29,4 @@
                  iyy="${1/12*0.08*(0.156**2+0.043**2)}" iyz="0.0"
                  izz="${1/12*0.08*(0.140**2+0.156**2)}" />
-        <!-- <inertia ixx="1.0" ixy="0.0" ixz="0.0"
-                 iyy="1.0" iyz="0.0"
-                 izz="1.0" /> -->
       </inertial>
     </link>
@@ -41,5 +36,5 @@
       <origin xyz="0.1560 0.0 0.0215" rpy="0.0 0.0 0.0 " />
       <axis xyz="0.0 -1.0 0.0 " />
-      <limit lower="${-M_PI/2}" upper="${M_PI/2}" effort="10" velocity="10" />
+      <limit lower="${-M_PI/2}" upper="${M_PI/2}" effort="25" velocity="11.031179004" />
       <!-- <dynamics damping="0.2" friction="0" /> -->
     </joint>
@@ -54,8 +49,6 @@
       <collision>
         <origin xyz="${0.1166/2+0.0224} 0.0 0.0" rpy="0.0 0.0 0.0" />
-        <!-- <origin xyz="0.0 0.0 0.0" rpy="${M_PI/2} 0.0 ${M_PI/2}" /> -->
         <geometry>
           <box size="0.1166 0.124 0.043" />
-          <!-- <mesh filename="package://sobit_pro_description/meshes/arm/arm_upper.stl" scale="0.001 0.001 0.001" /> -->
         </geometry>
       </collision>
@@ -66,7 +59,4 @@
                  iyy="${1/12*0.08*(0.124**2 +0.043**2)}" iyz="0.0"
                  izz="${1/12*0.08*(0.1166**2+0.124**2)}" />
-        <!-- <inertia ixx="1.0" ixy="0.0" ixz="0.0"
-                 iyy="1.0" iyz="0.0"
-                 izz="1.0" /> -->
       </inertial>
     </link>
@@ -77,5 +67,5 @@
       <axis xyz="0.0 1.0 0.0 " />
       <mimic joint="${prefix}_shoulder_1_tilt_joint" multiplier="1" offset="0" />
-      <limit lower="${-M_PI/2}" upper="${M_PI/2}" effort="10" velocity="10" />
+      <limit lower="${-M_PI/2}" upper="${M_PI/2}" effort="25" velocity="11.031179004" />
       <!-- <dynamics damping="0.2" friction="0" /> -->
     </joint>
@@ -86,5 +76,5 @@
       <origin xyz="0.1500 0.0 0.0" rpy="0.0 0.0 0.0" />
       <axis xyz="0.0 -1.0 0.0 " />
-      <limit lower="${-M_PI/2}" upper="${M_PI/2}" effort="10" velocity="10" />
+      <limit lower="${-M_PI/2}" upper="${M_PI/2}" effort="25" velocity="9.59233" />
       <!-- <dynamics damping="0.2" friction="0" /> -->
     </joint>
@@ -99,8 +89,6 @@
       <collision>
         <origin xyz="${0.023+0.127/2} 0.0 0.0" rpy="0.0 0.0 0.0" />
-        <!-- <origin xyz="0.0 0.0 0.0" rpy="${M_PI/2} 0.0 ${M_PI/2}" /> -->
         <geometry>
           <box size="0.127 0.048 0.035" />
-          <!-- <mesh filename="package://sobit_pro_description/meshes/arm/arm_inner.stl" scale="0.001 0.001 0.001" /> -->
         </geometry>
       </collision>
@@ -111,7 +99,4 @@
                  iyy="${1/12*0.08*(0.048**2+0.035**2)}" iyz="0.0"
                  izz="${1/12*0.08*(0.127**2+0.048**2)}" />
-        <!-- <inertia ixx="1.0" ixy="0.0" ixz="0.0"
-                 iyy="1.0" iyz="0.0"
-                 izz="1.0" /> -->
       </inertial>
     </link>
@@ -122,5 +107,5 @@
       <axis xyz="0.0 1.0 0.0 " />
       <mimic joint="${prefix}_elbow_upper_1_tilt_joint" multiplier="1" offset="0" />
-      <limit lower="${-M_PI/2}" upper="${M_PI/2}" effort="10" velocity="10" />
+      <limit lower="${-M_PI/2}" upper="${M_PI/2}" effort="25" velocity="9.59233" />
       <!-- <dynamics damping="0.2" friction="0" /> -->
     </joint>
@@ -131,5 +116,5 @@
       <origin xyz="0.1500 0.0 0.0" rpy="0.0 0.0 0.0" />
       <axis xyz="0.0 -1.0 0.0 " />
-      <limit lower="${-M_PI/2}" upper="${M_PI/2}" effort="10" velocity="10" />
+      <limit lower="${-M_PI/2}" upper="${M_PI/2}" effort="25" velocity="4.796165" />
       <!-- <dynamics damping="0.2" friction="0" /> -->
     </joint>
@@ -144,8 +129,6 @@
       <collision>
         <origin xyz="${0.028-0.005/2} 0.0 -${(0.0215-0.01825)/2}" rpy="0.0 0.0 0.0" />
-        <!-- <origin xyz="0.0 0.0 0.0" rpy="${M_PI/2} 0.0 ${M_PI/2}" /> -->
         <geometry>
           <box size="0.005 0.041 0.024" />
-          <!-- <mesh filename="package://sobit_pro_description/meshes/arm/arm_elbow_lower_tilt.stl" scale="0.001 0.001 0.001" /> -->
         </geometry>
       </collision>
@@ -156,7 +139,4 @@
                  iyy="${1/12*0.08*(0.041**2+0.024**2)}" iyz="0.0"
                  izz="${1/12*0.08*(0.005**2+0.041**2)}" />
-        <!-- <inertia ixx="1.0" ixy="0.0" ixz="0.0"
-                 iyy="1.0" iyz="0.0"
-                 izz="1.0" /> -->
       </inertial>
     </link>
@@ -166,5 +146,5 @@
       <origin xyz="0.028 0.0 0.0" rpy="0.0 0.0 0.0" />
       <axis xyz="1.0 0.0 0.0 " />
-      <limit lower="${-M_PI/2}" upper="${M_PI/2}" effort="10" velocity="10" />
+      <limit lower="${-M_PI/2}" upper="${M_PI/2}" effort="25" velocity="4.796165" />
       <!-- <dynamics damping="0.2" friction="0" /> -->
     </joint>
@@ -179,8 +159,6 @@
       <collision>
         <origin xyz="${0.002+0.120/2} 0.0 -${(0.0215-0.01825)/2}" rpy="0.0 0.0 0.0" />
-        <!-- <origin xyz="0.0 0.0 0.0" rpy="${M_PI/2} 0.0 ${M_PI/2}" /> -->
         <geometry>
           <box size="0.120 0.048 0.03975" />
-          <!-- <mesh filename="package://sobit_pro_description/meshes/arm/arm_elbow_lower_pan.stl" scale="0.001 0.001 0.001" /> -->
         </geometry>
       </collision>
@@ -188,11 +166,7 @@
         <origin xyz="${0.002+0.120/2} 0.0 -${(0.0215-0.01825)/2}" rpy="0.0 0.0 ${M_PI/2}" />
         <mass value="0.08" />
-        <!-- CHECK -->
         <inertia ixx="${1/12*0.08*(0.120**2+0.03975**2)}" ixy="0.0" ixz="0.0"
                  iyy="${1/12*0.08*(0.048**2+0.03975**2)}" iyz="0.0"
                  izz="${1/12*0.08*(0.120**2+0.048**2)}" />
-        <!-- <inertia ixx="0.001" ixy="0.0" ixz="0.0"
-                 iyy="0.001" iyz="0.0"
-                 izz="0.001" /> -->
       </inertial>
     </link>
@@ -202,5 +176,5 @@
       <origin xyz="0.122009 0.0 0.0" rpy="0.0 0.0 0.0" />
       <axis xyz="0.0 -1.0 0.0" />
-      <limit lower="${-M_PI/2}" upper="${M_PI/2}" effort="10" velocity="10" />
+      <limit lower="${-M_PI/2}" upper="${M_PI/2}" effort="25" velocity="4.796165" />
       <!-- <dynamics damping="0.2" friction="0" /> -->
     </joint>

File: sobit_pro_description/urdf/hand/hand.urdf.xacro (robot description, xacro)
@@ -19,8 +19,6 @@
       <collision>
         <origin xyz="${0.0215+(0.08251-0.0215)/2} 0.0 ${(0.0415-0.033)/2}" rpy="0.0 0.0 0.0" />
-        <!-- <origin xyz="0.0 0.0 0.0" rpy="${M_PI/2.0} 0.0 ${M_PI/2.0}" /> -->
         <geometry>
           <box size="0.06102 0.102 0.0745" />
-          <!-- <mesh filename="package://sobit_pro_description/meshes/hand/hand_base.stl" scale="0.001 0.001 0.001" /> -->
         </geometry>
       </collision>
@@ -31,18 +29,7 @@
                  iyy="${1/12*0.08*(0.102**2  +0.0745**2)}" iyz="0.0"
                  izz="${1/12*0.08*(0.06102**2+0.102**2)}" />
-        <!-- <inertia ixx="1.0" ixy="0.0" ixz="0.0"
-                 iyy="1.0" iyz="0.0"
-                 izz="1.0" /> -->
-      </inertial>
-    </link>
-    <!-- <joint name="${prefix_hand}_joint" type="revolute">
-      <parent link="${prefix_hand}_base_link" />
-      <child link="${prefix_hand}_link" />
-      <origin xyz="0.0631932 -0.0151495 0.0222231" rpy="0.0 0.0 0.0" />
-      <axis xyz="0.0 0.0 1.0" />
-      <limit lower="${-M_PI/2.0}" upper="0" effort="1" velocity="1" />
-    </joint>
-    <link name="${prefix_hand}_link" /> -->
-    <joint name="${prefix_hand}_inner_l_joint" type="revolute">
+      </inertial>
+    </link>
+    <joint name="${prefix_hand}_inner_l_joint" type="continuous">
       <parent link="${prefix_hand}_base_link" />
       <child link="${prefix_hand}_inner_l_link" />
@@ -50,5 +37,4 @@
       <axis xyz="0.0 0.0 1.0" />
       <mimic joint="${prefix_hand}_joint" multiplier="-1.0" offset="0" />
-      <limit lower="${-M_PI/2.0}" upper="0" effort="1" velocity="1" />
     </joint>
     <link name="${prefix_hand}_inner_l_link">
@@ -62,8 +48,6 @@
       <collision>
         <origin xyz="${0.05408+(0.06006-0.00707)/2} 0.0 -${0.066/2}" rpy="0.0 0.0 0.0" />
-        <!-- <origin xyz="0.0 0.0 0.0" rpy="0.0 0.0 ${M_PI/2.0}" /> -->
         <geometry>
           <box size="${0.06006-0.0071} 0.01 0.066" />
-          <!-- <mesh filename="package://sobit_pro_description/meshes/hand/hand_inner_l.stl" scale="0.001 0.001 0.001" /> -->
         </geometry>
       </collision>
@@ -74,7 +58,4 @@
                  iyy="${1/12*0.08*(0.01**2+0.066**2)}"             iyz="0.0"
                  izz="${1/12*0.08*((0.06006-0.0071)**2+0.01**2)}" />
-        <!-- <inertia ixx="1.0" ixy="0.0" ixz="0.0"
-                 iyy="1.0" iyz="0.0"
-                 izz="1.0" /> -->
       </inertial>
     </link>
@@ -84,6 +65,5 @@
       <origin xyz="0.0631932 -0.0151495 0.0372231" rpy="0.0 0.0 0.0" />
       <axis xyz="0.0 0.0 1.0" />
-      <!-- <mimic joint="${prefix_hand}_joint" multiplier="1.0" offset="0" /> -->
-      <limit lower="${-M_PI/2.0}" upper="0" effort="1" velocity="1" />
+      <limit lower="${-M_PI/2.0}" upper="0" effort="25" velocity="4.796165" />
     </joint>
     <link name="${prefix_hand}_link">
@@ -97,8 +77,6 @@
       <collision>
         <origin xyz="${0.05408+(0.06006-0.00707)/2} 0.0 -${0.066/2}" rpy="0.0 0.0 0.0" />
-        <!-- <origin xyz="0.0 0.0 0.0" rpy="0.0 0.0 ${M_PI/2.0}" /> -->
         <geometry>
           <box size="${0.06006-0.0071} 0.01 0.066" />
-          <!-- <mesh filename="package://sobit_pro_description/meshes/hand/hand_inner_r.stl" scale="0.001 0.001 0.001" /> -->
         </geometry>
       </collision>
@@ -109,18 +87,12 @@
                  iyy="${1/12*0.08*(0.01**2+0.066**2)}"             iyz="0.0"
                  izz="${1/12*0.08*((0.06006-0.0071)**2+0.01**2)}" />
-        <!-- <inertia ixx="1.0" ixy="0.0" ixz="0.0"
-                 iyy="1.0" iyz="0.0"
-                 izz="1.0" /> -->
-      </inertial>
-    </link>
-    <joint name="${prefix_hand}_outer_l_joint" type="revolute">
-      <!-- <parent link="${prefix_hand}_inner_l_link" /> -->
+      </inertial>
+    </link>
+    <joint name="${prefix_hand}_outer_l_joint" type="continuous">
       <parent link="${prefix_hand}_base_link" />
       <child link="${prefix_hand}_outer_l_link" />
-      <!-- <origin xyz="-0.01988747 0.025 -0.01022197" rpy="0.0 0.0 0.0" /> -->
       <origin xyz="0.043193 0.04015 0.0282231" rpy="0.0 0.0 0.0" />
       <axis xyz="0.0 0.0 1.0" />
       <mimic joint="${prefix_hand}_inner_l_joint" multiplier="1.0" offset="0" />
-      <limit lower="${-M_PI/2.0}" upper="0" effort="1" velocity="1" />
     </joint>
     <link name="${prefix_hand}_outer_l_link">
@@ -134,8 +106,6 @@
       <collision>
         <origin xyz="${0.06123+0.04281/2} 0.0 -${0.056/2}" rpy="0.0 0.0 0.0" />
-        <!-- <origin xyz="0.0 0.0 0.0" rpy="0.0 0.0 ${M_PI/2.0}" /> -->
         <geometry>
           <box size="0.04281 0.01 0.056" />
-          <!-- <mesh filename="package://sobit_pro_description/meshes/hand/hand_outer_l.stl" scale="0.001 0.001 0.001" /> -->
         </geometry>
       </collision>
@@ -146,18 +116,12 @@
                  iyy="${1/12*0.08*(0.01**2   +0.056**2)}" iyz="0.0"
                  izz="${1/12*0.08*(0.04281**2+0.01**2)}" />
-        <!-- <inertia ixx="1.0" ixy="0.0" ixz="0.0"
-                 iyy="1.0" iyz="0.0"
-                 izz="1.0" /> -->
-      </inertial>
-    </link>
-    <joint name="${prefix_hand}_outer_r_joint" type="revolute">
-      <!-- <parent link="${prefix_hand}_inner_r_link" /> -->
+      </inertial>
+    </link>
+    <joint name="${prefix_hand}_outer_r_joint" type="continuous">
       <parent link="${prefix_hand}_base_link" />
       <child link="${prefix_hand}_outer_r_link" />
-      <!-- <origin xyz="-0.01988747 -0.025 -0.01022197" rpy="0.0 0.0 0.0" /> -->
       <origin xyz="0.043193 -0.04015 0.0282231" rpy="0.0 0.0 0.0" />
       <axis xyz="0.0 0.0 1.0" />
       <mimic joint="${prefix_hand}_joint" multiplier="1.0" offset="0" />
-      <limit lower="${-M_PI/2.0}" upper="0" effort="1" velocity="1" />
     </joint>
     <link name="${prefix_hand}_outer_r_link">
@@ -171,8 +135,6 @@
       <collision>
         <origin xyz="${0.06123+0.04281/2} 0.0 -${0.056/2}" rpy="0.0 0.0 0.0" />
-        <!-- <origin xyz="0.0 0.0 0.0" rpy="0.0 0.0 ${M_PI/2.0}" /> -->
         <geometry>
           <box size="0.04281 0.01 0.056" />
-          <!-- <mesh filename="package://sobit_pro_description/meshes/hand/hand_outer_r.stl" scale="0.001 0.001 0.001" /> -->
         </geometry>
       </collision>
@@ -183,10 +145,7 @@
                  iyy="${1/12*0.08*(0.01**2   +0.056**2)}" iyz="0.0"
                  izz="${1/12*0.08*(0.04281**2+0.01**2)}" />
-        <!-- <inertia ixx="1.0" ixy="0.0" ixz="0.0"
-                 iyy="1.0" iyz="0.0"
-                 izz="1.0" /> -->
-      </inertial>
-    </link>
-    <joint name="${prefix_hand}_${prefix_finger}_l_joint" type="revolute">
+      </inertial>
+    </link>
+    <joint name="${prefix_hand}_${prefix_finger}_l_joint" type="continuous">
       <parent link="${prefix_hand}_inner_l_link" />
       <child link="${prefix_hand}_${prefix_finger}_l_link" />
@@ -194,5 +153,4 @@
       <axis xyz="0.0 0.0 1.0" />
       <mimic joint="${prefix_hand}_joint" multiplier="1.0" offset="0" />
-      <limit lower="${-M_PI/2.0}" upper="0" effort="1" velocity="1" />
     </joint>
     <link name="${prefix_hand}_${prefix_finger}_l_link">
@@ -206,8 +164,6 @@
       <collision>
         <origin xyz="${0.007071+(0.012042+0.061128)/2} 0.0 -${0.018/2}" rpy="0.0 0.0 0.0" />
-        <!-- <origin xyz="0.0 0.0 0.0" rpy="0.0 0.0 ${M_PI/2.0}" /> -->
         <geometry>
           <box size="${0.012042+0.061128} 0.01137 0.044" />
-          <!-- <mesh filename="package://sobit_pro_description/meshes/hand/hand_finger_l.stl" scale="0.001 0.001 0.001" /> -->
         </geometry>
       </collision>
@@ -218,10 +174,7 @@
                  iyy="${1/12*0.08*(0.01137**2+0.044**2)}"             iyz="0.0"
                  izz="${1/12*0.08*((0.012042+0.061128)**2+0.01137**2)}" />
-        <!-- <inertia ixx="1.0" ixy="0.0" ixz="0.0"
-                 iyy="1.0" iyz="0.0"
-                 izz="1.0" /> -->
-      </inertial>
-    </link>
-    <joint name="${prefix_hand}_${prefix_finger}_r_joint" type="revolute">
+      </inertial>
+    </link>
+    <joint name="${prefix_hand}_${prefix_finger}_r_joint" type="continuous">
       <parent link="${prefix_hand}_link" />
       <child link="${prefix_hand}_${prefix_finger}_r_link" />
@@ -229,5 +182,4 @@
       <axis xyz="0.0 0.0 1.0" />
       <mimic joint="${prefix_hand}_joint" multiplier="-1.0" offset="0" />
-      <limit lower="${-M_PI/2.0}" upper="0" effort="1" velocity="1" />
     </joint>
     <link name="${prefix_hand}_${prefix_finger}_r_link">
@@ -241,8 +193,6 @@
       <collision>
         <origin xyz="${0.007071+(0.012042+0.061128)/2} 0.0 -${0.018/2}" rpy="0.0 0.0 0.0" />
-        <!-- <origin xyz="0.0 0.0 0.0" rpy="0.0 0.0 ${M_PI/2.0}" /> -->
         <geometry>
           <box size="${0.012042+0.061128} 0.01137 0.044" />
-          <!-- <mesh filename="package://sobit_pro_description/meshes/hand/hand_finger_r.stl" scale="0.001 0.001 0.001" /> -->
         </geometry>
       </collision>
@@ -253,7 +203,4 @@
                  iyy="${1/12*0.08*(0.01137**2+0.044**2)}"               iyz="0.0"
                  izz="${1/12*0.08*((0.012042+0.061128)**2+0.01137**2)}" />
-        <!-- <inertia ixx="1.0" ixy="0.0" ixz="0.0"
-                 iyy="1.0" iyz="0.0"
-                 izz="1.0" /> -->
       </inertial>
     </link>

File: sobit_pro_description/urdf/head/head.urdf.xacro (robot description, xacro)
@@ -5,12 +5,9 @@
   <xacro:macro name="head" params="prefix parent">
     <joint name="${prefix}_base_joint" type="fixed">
-    <!-- <joint name="${prefix}_camera_base_joint" type="fixed"> -->
       <parent link="${parent}" />
-      <!-- <child link="${prefix}_camera_base_link" /> -->
       <child link="${prefix}_base_link" />
       <origin xyz="0.0900 0.0 0.5270" rpy="0.0 0.0 0.0" />
     </joint>
     <link name="${prefix}_base_link">
-    <!-- <link name="${prefix}_camera_base_link"> -->
       <visual>
         <origin xyz="0.0 0.0 0.0" rpy="${M_PI/2.0} 0.0 ${M_PI/2.0}" />
@@ -22,8 +19,6 @@
       <collision>
         <origin xyz="${0.05125-0.15125/2} 0.0 0.0" rpy="0.0 0.0 0.0" />
-        <!-- <origin xyz="0.0 0.0 0.0" rpy="${M_PI/2.0} 0.0 ${M_PI/2.0}" /> -->
         <geometry>
           <box size="0.15125 0.0285 0.044"/>
-          <!-- <mesh filename="package://sobit_pro_description/meshes/head/head_camera_base.stl" scale="0.001 0.001 0.001" /> -->
         </geometry>
       </collision>
@@ -34,21 +29,14 @@
                  iyy="${1/12*0.08*(0.0285**2 +0.044**2)}" iyz="0.0"
                  izz="${1/12*0.08*(0.15125**2+0.0285**2)}" />
-        <!-- <inertia ixx="1.0" ixy="0.0" ixz="0.0"
-                 iyy="1.0" iyz="0.0"
-                 izz="1.0" /> -->
       </inertial>
     </link>
-    <!-- <joint name="${prefix}_camera_pan_joint" type="revolute"> -->
     <joint name="${prefix}_pan_joint" type="revolute">
       <parent link="${prefix}_base_link" />
-      <!-- <parent link="${prefix}_camera_base_link" /> -->
       <child link="${prefix}_pan_link" />
-      <!-- <child link="${prefix}_camera_pan_link" /> -->
       <origin xyz="0.03985 0.0 0.0190" rpy="0.0 0.0 0.0" />
       <axis xyz="0 0 1" />
-      <limit effort="30" lower="${-M_PI/2.0}" upper="${M_PI/2.0}" velocity="${M_PI/2.0}" />
+      <limit effort="25" lower="${-M_PI/2.0}" upper="${M_PI/2.0}" velocity="${M_PI/2.0}" />
     </joint>
     <link name="${prefix}_pan_link">
-    <!-- <link name="${prefix}_camera_pan_link"> -->
       <visual>
         <origin xyz="0.0 0.0 0.0" rpy="0.0 0.0 ${M_PI/2.0}" />
@@ -60,8 +48,6 @@
       <collision>
         <origin xyz="0.0 0.0 ${0.00525+0.03525/2}" rpy="0.0 0.0 0.0" />
-        <!-- <origin xyz="0.0 0.0 0.0" rpy="0.0 0.0 ${M_PI/2.0}" /> -->
         <geometry>
           <box size="0.0285 0.037 0.03525"/>
-          <!-- <mesh filename="package://sobit_pro_description/meshes/head/head_camera_pan.stl" scale="0.001 0.001 0.001" /> -->
         </geometry>
       </collision>
@@ -72,21 +58,14 @@
                  iyy="${1/12*0.08*(0.037**2 +0.03525**2)}" iyz="0.0"
                  izz="${1/12*0.08*(0.0285**2+0.037**2)}" />
-        <!-- <inertia ixx="1.0" ixy="0.0" ixz="0.0"
-                 iyy="1.0" iyz="0.0"
-                 izz="1.0" /> -->
       </inertial>
     </link>
     <joint name="${prefix}_tilt_joint" type="revolute">
-    <!-- <joint name="${prefix}_camera_tilt_joint" type="revolute"> -->
       <parent link="${prefix}_pan_link" />
-      <!-- <parent link="${prefix}_camera_pan_link" /> -->
       <child link="${prefix}_tilt_link" />
-      <!-- <child link="${prefix}_camera_tilt_link" /> -->
       <origin xyz="0.0 0.0 0.0405" rpy="0.0 0.0 0.0" />
       <axis xyz="0 -1 0" />
-      <limit effort="30" lower="${-M_PI/2.0}" upper="${M_PI/2.0}" velocity="${M_PI/2.0}" />
+      <limit effort="25" lower="${-M_PI/2.0}" upper="${M_PI/2.0}" velocity="${M_PI/2.0}" />
     </joint>
     <link name="${prefix}_tilt_link">
-    <!-- <link name="${prefix}_camera_tilt_link"> -->
       <visual>
         <origin xyz="0.0 0.0 0.0" rpy="0.0 0.0 ${M_PI/2.0}" />
@@ -98,8 +77,6 @@
       <collision>
         <origin xyz="0.0 0.0 ${0.028+0.0115/2}" rpy="0.0 0.0 0.0" />
-        <!-- <origin xyz="0.0 0.0 0.0" rpy="0.0 0.0 ${M_PI/2.0}" /> -->
         <geometry>
           <box size="0.046 0.0466 0.0115"/>
-          <!-- <mesh filename="package://sobit_pro_description/meshes/head/head_camera_tilt.stl" scale="0.001 0.001 0.001" /> -->
         </geometry>
       </collision>
@@ -110,7 +87,4 @@
                  iyy="${1/12*0.08*(0.0466**2+0.0115**2)}" iyz="0.0"
                  izz="${1/12*0.08*(0.046**2 +0.0466**2)}" />
-        <!-- <inertia ixx="1.0" ixy="0.0" ixz="0.0"
-                 iyy="1.0" iyz="0.0"
-                 izz="1.0" /> -->
       </inertial>
     </link>
