Commit message: [UPD] velocities and effort limits are updated based on real robot

File: sobit_pro_description/urdf/wheel/wheel.urdf.xacro (robot description, xacro)
@@ -19,20 +19,14 @@
       <collision>
         <origin xyz="${0.01388-0.05525/2} 0.0 -${0.005+0.034/2+0.02/2}" rpy="0.0 0.0 0.0" />
-        <!-- <origin xyz="0.0 0.0 0.0" rpy="${M_PI/2.0} 0.0 ${M_PI/2.0}" /> -->
         <geometry>
           <box size="0.05525 0.0285 0.084" />
-          <!-- <mesh filename="package://sobit_pro_description/meshes/wheel/wheel_base.stl" scale="0.001 0.001 0.001" /> -->
         </geometry>
       </collision>
       <inertial>
         <origin xyz="${0.01388-0.05525/2} 0.0 -${0.005+0.034/2+0.02/2}" rpy="0.0 0.0 0.0" />
-        <!-- <origin xyz="0.0 0.0 0.0" rpy="${M_PI/2.0} 0.0 ${M_PI/2.0}" /> -->
         <mass value="1" />
         <inertia ixx="${1/12*1*(0.05525**2+0.084**2)}" ixy="0.0" ixz="0.0"
                  iyy="${1/12*1*(0.0285**2 +0.084**2)}" iyz="0.0"
                  izz="${1/12*1*(0.05525**2+0.0285**2)}" />
-        <!-- <inertia ixx="1.0" ixy="0.0" ixz="0.0"
-                 iyy="1.0" iyz="0.0"
-                 izz="1.0" /> -->
       </inertial>
     </link>
@@ -44,5 +38,5 @@
       <child link="wheel_${prefix}_steer_link" />
       <axis xyz="0.0 0.0 1.0 " />
-      <limit lower="${-M_PI / 2}" upper="${M_PI/2}" effort="10" velocity="10" />
+      <limit lower="${-M_PI/2}" upper="${M_PI/2}" effort="25" velocity="4.796165" />
       <!-- <dynamics damping="0.2" friction="0" /> -->
     </joint>
@@ -57,9 +51,6 @@
       <collision>
         <origin xyz="${0.0244+0.0436/2} 0.0 ${0.034/2+0.0149-0.1766/2}" rpy="0.0 0.0 0.0" />
-        <!-- <origin xyz="0.0 0.0 0.0" rpy="${M_PI/2} 0.0 ${M_PI/2}" /> -->
         <geometry>
-          <!-- <box size="0.0495 0.1766 0.0436" /> -->
           <box size="0.0436 0.0495 0.1766" />
-          <!-- <mesh filename="package://sobit_pro_description/meshes/wheel/wheel_steer.stl" scale="0.001 0.001 0.001" /> -->
         </geometry>
       </collision>
@@ -70,7 +61,4 @@
                  iyy="${1/12*1*(0.0495**2+0.1766**2)}" iyz="0.0"
                  izz="${1/12*1*(0.0436**2+0.0495**2)}" />
-        <!-- <inertia ixx="1.0" ixy="0.0" ixz="0.0"
-                 iyy="1.0" iyz="0.0"
-                 izz="1.0" /> -->
       </inertial>
     </link>
@@ -82,5 +70,5 @@
       <child link="wheel_${prefix}_drive_link" />
       <axis xyz="-1.0 0.0 0.0 " />
-      <limit effort="10" velocity="10" />
+      <limit effort="25" velocity="7.913672" />
     </joint>
     <link name="wheel_${prefix}_drive_link">
@@ -94,8 +82,6 @@
       <collision>
         <origin xyz="-${0.0055+0.029/2} 0.0 0.0" rpy="${M_PI/2} 0.0 ${M_PI+M_PI/2.0}" />
-        <!-- <origin xyz="0.0 0.0 0.0" rpy="${M_PI/2} 0.0 ${M_PI+M_PI/2.0}" /> -->
         <geometry>
           <cylinder radius="${0.144/2}" length="0.029"/>
-          <!-- <mesh filename="package://sobit_pro_description/meshes/wheel/wheel_drive.stl" scale="0.001 0.001 0.001" /> -->
         </geometry>
       </collision>
@@ -106,7 +92,4 @@
                  iyy="${1/12*1*(3*(0.144/2)**2+0.029**2)}" iyz="0.0"
                  izz="${1/12*1*(3*(0.144/2)**2+0.029**2)}" />
-        <!-- <inertia ixx="1.0" ixy="0.0" ixz="0.0"
-                 iyy="1.0" iyz="0.0"
-                 izz="1.0" /> -->
       </inertial>
     </link>
@@ -125,5 +108,5 @@
     <xacro:stack_wheel_drive parent="wheel_b_r_steer_link" prefix="b_r" number="3" x_loc= "0.02" y_loc= "0.0" z_loc="-0.118" />
     <xacro:stack_wheel_drive parent="wheel_f_r_steer_link" prefix="f_r" number="4" x_loc= "0.02" y_loc= "0.0" z_loc="-0.118" />
-    <!-- <xacro:wheel_transmission prefix="${prefix}" /> -->
+    <xacro:wheel_transmission prefix="${prefix}" />
   </xacro:macro>
 </robot>

Commit message: [UPD] effort values

File: sobit_pro_description/urdf/arm/arm.urdf.xacro (robot description, xacro)
@@ -36,5 +36,5 @@
       <origin xyz="0.1560 0.0 0.0215" rpy="0.0 0.0 0.0 " />
       <axis xyz="0.0 -1.0 0.0 " />
-      <limit lower="${-M_PI/2}" upper="${M_PI/2}" effort="25" velocity="11.031179004" />
+      <limit lower="${-M_PI/2}" upper="${M_PI/2}" effort="${10.6*2}" velocity="11.031179004" />
       <!-- <dynamics damping="0.2" friction="0" /> -->
     </joint>
@@ -67,6 +67,6 @@
       <axis xyz="0.0 1.0 0.0 " />
       <mimic joint="${prefix}_shoulder_1_tilt_joint" multiplier="1" offset="0" />
-      <limit lower="${-M_PI/2}" upper="${M_PI/2}" effort="25" velocity="11.031179004" />
-      <!-- <dynamics damping="0.2" friction="0" /> -->
+      <limit lower="${-M_PI/2}" upper="${M_PI/2}" effort="${10.6*2}" velocity="11.031179004" />
+      <dynamics damping="0.2" friction="0" />
     </joint>
     <link name="${prefix}_shoulder_2_tilt_link" />
@@ -76,5 +76,5 @@
       <origin xyz="0.1500 0.0 0.0" rpy="0.0 0.0 0.0" />
       <axis xyz="0.0 -1.0 0.0 " />
-      <limit lower="${-M_PI/2}" upper="${M_PI/2}" effort="25" velocity="9.59233" />
+      <limit lower="${-M_PI/2}" upper="${M_PI/2}" effort="${4.1*2}" velocity="9.59233" />
       <!-- <dynamics damping="0.2" friction="0" /> -->
     </joint>
@@ -107,6 +107,6 @@
       <axis xyz="0.0 1.0 0.0 " />
       <mimic joint="${prefix}_elbow_upper_1_tilt_joint" multiplier="1" offset="0" />
-      <limit lower="${-M_PI/2}" upper="${M_PI/2}" effort="25" velocity="9.59233" />
-      <!-- <dynamics damping="0.2" friction="0" /> -->
+      <limit lower="${-M_PI/2}" upper="${M_PI/2}" effort="${4.1*2}" velocity="9.59233" />
+      <dynamics damping="0.2" friction="0" />
     </joint>
     <link name="${prefix}_elbow_upper_2_tilt_link" />
@@ -116,5 +116,5 @@
       <origin xyz="0.1500 0.0 0.0" rpy="0.0 0.0 0.0" />
       <axis xyz="0.0 -1.0 0.0 " />
-      <limit lower="${-M_PI/2}" upper="${M_PI/2}" effort="25" velocity="4.796165" />
+      <limit lower="${-M_PI/2}" upper="${M_PI/2}" effort="4.1" velocity="4.796165" />
       <!-- <dynamics damping="0.2" friction="0" /> -->
     </joint>
@@ -146,5 +146,5 @@
       <origin xyz="0.028 0.0 0.0" rpy="0.0 0.0 0.0" />
       <axis xyz="1.0 0.0 0.0 " />
-      <limit lower="${-M_PI/2}" upper="${M_PI/2}" effort="25" velocity="4.796165" />
+      <limit lower="${-M_PI/2}" upper="${M_PI/2}" effort="4.1" velocity="4.796165" />
       <!-- <dynamics damping="0.2" friction="0" /> -->
     </joint>
@@ -176,5 +176,5 @@
       <origin xyz="0.122009 0.0 0.0" rpy="0.0 0.0 0.0" />
       <axis xyz="0.0 -1.0 0.0" />
-      <limit lower="${-M_PI/2}" upper="${M_PI/2}" effort="25" velocity="4.796165" />
+      <limit lower="${-M_PI/2}" upper="${M_PI/2}" effort="4.1" velocity="4.796165" />
       <!-- <dynamics damping="0.2" friction="0" /> -->
     </joint>

File: sobit_pro_description/urdf/hand/hand.urdf.xacro (robot description, xacro)
@@ -65,5 +65,5 @@
       <origin xyz="0.0631932 -0.0151495 0.0372231" rpy="0.0 0.0 0.0" />
       <axis xyz="0.0 0.0 1.0" />
-      <limit lower="${-M_PI/2.0}" upper="0" effort="25" velocity="4.796165" />
+      <limit lower="${-M_PI/2.0}" upper="0" effort="4.1" velocity="4.796165" />
     </joint>
     <link name="${prefix_hand}_link">

File: sobit_pro_description/urdf/head/head.urdf.xacro (robot description, xacro)
@@ -36,5 +36,5 @@
       <origin xyz="0.03985 0.0 0.0190" rpy="0.0 0.0 0.0" />
       <axis xyz="0 0 1" />
-      <limit effort="25" lower="${-M_PI/2.0}" upper="${M_PI/2.0}" velocity="${M_PI/2.0}" />
+      <limit lower="${-M_PI/2.0}" upper="${M_PI/2.0}" effort="4.1" velocity="4.796165" />
     </joint>
     <link name="${prefix}_pan_link">
@@ -65,5 +65,5 @@
       <origin xyz="0.0 0.0 0.0405" rpy="0.0 0.0 0.0" />
       <axis xyz="0 -1 0" />
-      <limit effort="25" lower="${-M_PI/2.0}" upper="${M_PI/2.0}" velocity="${M_PI/2.0}" />
+      <limit lower="${-M_PI/2.0}" upper="${M_PI/2.0}" effort="4.1" velocity="4.796165" />
     </joint>
     <link name="${prefix}_tilt_link">

File: sobit_pro_description/urdf/wheel/wheel.urdf.xacro (robot description, xacro)
@@ -38,5 +38,5 @@
       <child link="wheel_${prefix}_steer_link" />
       <axis xyz="0.0 0.0 1.0 " />
-      <limit lower="${-M_PI/2}" upper="${M_PI/2}" effort="25" velocity="4.796165" />
+      <limit lower="${-M_PI/2}" upper="${M_PI/2}" effort="4.1" velocity="4.796165" />
       <!-- <dynamics damping="0.2" friction="0" /> -->
     </joint>
@@ -70,5 +70,5 @@
       <child link="wheel_${prefix}_drive_link" />
       <axis xyz="-1.0 0.0 0.0 " />
-      <limit effort="25" velocity="7.913672" />
+      <limit effort="3.0" velocity="7.913672" />
     </joint>
     <link name="wheel_${prefix}_drive_link">
