Commit message: [UPD] update urdf versio

File: sobit_pro_sim_description/robots/sobit_pro.urdf (robot description, URDF)
Before this commit: robot sobit_pro, 64 links, 63 joints
Links:
- removed link arm_elbow_upper_2_tilt_link
- removed link arm_shoulder_2_tilt_link
Joints:
- removed joint arm_elbow_upper_2_tilt_joint
- removed joint arm_shoulder_2_tilt_joint
- joint arm_elbow_lower_pan_joint: limit lower=-1.570796326795 upper=1.570796326795 effort=10 velocity=10 -> lower=-1.570796326795 upper=1.570796326795 effort=4.1 velocity=4.796165
- joint arm_elbow_lower_tilt_joint: limit lower=-1.570796326795 upper=1.570796326795 effort=10 velocity=10 -> lower=-1.570796326795 upper=1.570796326795 effort=4.1 velocity=4.796165
- joint arm_elbow_upper_1_tilt_joint: limit lower=-1.570796326795 upper=1.570796326795 effort=10 velocity=10 -> lower=-1.570796326795 upper=1.570796326795 effort=8.2 velocity=9.59233
- joint arm_shoulder_1_tilt_joint: limit lower=-1.570796326795 upper=1.570796326795 effort=10 velocity=10 -> lower=-1.570796326795 upper=1.570796326795 effort=21.2 velocity=11.031179004
- joint arm_wrist_tilt_joint: limit lower=-1.570796326795 upper=1.570796326795 effort=10 velocity=10 -> lower=-1.570796326795 upper=1.570796326795 effort=4.1 velocity=4.796165
- joint hand_finger_l_joint: limit lower=-1.570796326795 upper=0 effort=1 velocity=1 -> (none); type revolute -> continuous
- joint hand_finger_r_joint: limit lower=-1.570796326795 upper=0 effort=1 velocity=1 -> (none); type revolute -> continuous
- joint hand_inner_l_joint: limit lower=-1.570796326795 upper=0 effort=1 velocity=1 -> (none); type revolute -> continuous
- joint hand_joint: limit lower=-1.570796326795 upper=0 effort=1 velocity=1 -> lower=-1.570796326795 upper=0 effort=4.1 velocity=4.796165
- joint hand_outer_l_joint: limit lower=-1.570796326795 upper=0 effort=1 velocity=1 -> (none); type revolute -> continuous
- joint hand_outer_r_joint: limit lower=-1.570796326795 upper=0 effort=1 velocity=1 -> (none); type revolute -> continuous
- joint head_pan_joint: limit lower=-1.570796326795 upper=1.570796326795 effort=30 velocity=1.570796326795 -> lower=-1.570796326795 upper=1.570796326795 effort=4.1 velocity=4.796165
- joint head_tilt_joint: limit lower=-1.570796326795 upper=1.570796326795 effort=30 velocity=1.570796326795 -> lower=-1.570796326795 upper=1.570796326795 effort=4.1 velocity=4.796165
- joint wheel_b_l_drive_joint: limit effort=10 velocity=10 -> effort=3.0 velocity=7.913672
- joint wheel_b_l_steer_joint: limit lower=-1.570796326795 upper=1.570796326795 effort=10 velocity=10 -> lower=-1.570796326795 upper=1.570796326795 effort=4.1 velocity=4.796165
- joint wheel_b_r_drive_joint: limit effort=10 velocity=10 -> effort=3.0 velocity=7.913672
- joint wheel_b_r_steer_joint: limit lower=-1.570796326795 upper=1.570796326795 effort=10 velocity=10 -> lower=-1.570796326795 upper=1.570796326795 effort=4.1 velocity=4.796165
- joint wheel_f_l_drive_joint: limit effort=10 velocity=10 -> effort=3.0 velocity=7.913672
- joint wheel_f_l_steer_joint: limit lower=-1.570796326795 upper=1.570796326795 effort=10 velocity=10 -> lower=-1.570796326795 upper=1.570796326795 effort=4.1 velocity=4.796165
- joint wheel_f_r_drive_joint: limit effort=10 velocity=10 -> effort=3.0 velocity=7.913672
- joint wheel_f_r_steer_joint: limit lower=-1.570796326795 upper=1.570796326795 effort=10 velocity=10 -> lower=-1.570796326795 upper=1.570796326795 effort=4.1 velocity=4.796165
