Commit message: [[ADD] add sobit pro urdf model for isaac sim

File: sobit_pro_sim_description/robots/sobit_pro_isaac.urdf (robot description, URDF)
Before this commit: robot sobit_pro, 62 links, 61 joints
Links:
- link arm_base_link: geometry collision box size=0.140 0.156 0.043; visual mesh filename=package://sobit_pro/sobit_pro_description/meshes/arm/arm_ba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 scale=0.001 0.001 0.001
- link arm_elbow_lower_pan_link: geometry collision box size=0.120 0.048 0.03975; visual mesh filename=package://sobit_pro/sobit_pro_description/meshes/arm/arm_el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 scale=0.001 0.001 0.001
- link arm_elbow_lower_tilt_link: geometry collision box size=0.005 0.041 0.024; visual mesh filename=package://sobit_pro/sobit_pro_description/meshes/arm/arm_el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 scale=0.001 0.001 0.001
- link arm_elbow_upper_1_tilt_link: geometry collision box size=0.127 0.048 0.035; visual mesh filename=package://sobit_pro/sobit_pro_description/meshes/arm/arm_in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 scale=0.001 0.001 0.001
- link arm_shoulder_1_tilt_link: geometry collision box size=0.1166 0.124 0.043; visual mesh filename=package://sobit_pro/sobit_pro_description/meshes/arm/arm_up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 scale=0.001 0.001 0.001
- link back_base_link: geometry collision box size=0.02 0.02 0.517; visual mesh filename=package://sobit_pro/sobit_pro_description/meshes/back/back_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 scale=0.001 0.001 0.001
- link cover_link: geometry collision box size=0.35786 0.3965 0.489; visual mesh filename=package://sobit_pro/sobit_pro_description/meshes/body/cover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 scale=0.001 0.001 0.001
- link hand_base_link: geometry collision box size=0.06102 0.102 0.0745; visual mesh filename=package://sobit_pro/sobit_pro_description/meshes/hand/hand_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 scale=0.001 0.001 0.001
- link hand_camera_link: geometry collision box size=0.023 0.042 0.042; visual mesh filename=package://realsense_ros/realsense2_description/meshes/d405.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
- link hand_finger_l_link: geometry collision box size=0.07317 0.01137 0.044; visual mesh filename=package://sobit_pro/sobit_pro_description/meshes/hand/hand_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 scale=0.001 0.001 0.001
- link hand_finger_r_link: geometry collision box size=0.07317 0.01137 0.044; visual mesh filename=package://sobit_pro/sobit_pro_description/meshes/hand/hand_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 scale=0.001 0.001 0.001
- link hand_inner_l_link: geometry collision box size=0.05296 0.01 0.066; visual mesh filename=package://sobit_pro/sobit_pro_description/meshes/hand/hand_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 scale=0.001 0.001 0.001
- link hand_link: geometry collision box size=0.05296 0.01 0.066; visual mesh filename=package://sobit_pro/sobit_pro_description/meshes/hand/hand_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 scale=0.001 0.001 0.001
- link hand_outer_l_link: geometry collision box size=0.04281 0.01 0.056; visual mesh filename=package://sobit_pro/sobit_pro_description/meshes/hand/hand_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 scale=0.001 0.001 0.001
- link hand_outer_r_link: geometry collision box size=0.04281 0.01 0.056; visual mesh filename=package://sobit_pro/sobit_pro_description/meshes/hand/hand_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 scale=0.001 0.001 0.001
- link head_base_link: geometry collision box size=0.15125 0.0285 0.044; visual mesh filename=package://sobit_pro/sobit_pro_description/meshes/head/head_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 scale=0.001 0.001 0.001
- link head_pan_link: geometry collision box size=0.0285 0.037 0.03525; visual mesh filename=package://sobit_pro/sobit_pro_description/meshes/head/head_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 scale=0.001 0.001 0.001
- link head_tilt_link: geometry collision box size=0.046 0.0466 0.0115; visual mesh filename=package://sobit_pro/sobit_pro_description/meshes/head/head_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 scale=0.001 0.001 0.001
- link lidar_base_link: geometry collision box size=0.092 0.184 0.007; visual mesh filename=package://sobit_pro/sobit_pro_description/meshes/sensor/lid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 scale=0.001 0.001 0.001
- link mic_base_link: geometry collision box size=0.0292 0.12919999999999998 0.03; visual mesh filename=package://sobit_pro/sobit_pro_description/meshes/sensor/mic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 scale=0.001 0.001 0.001
- link mic_link: geometry collision cylinder length=0.281 radius=0.011; visual mesh filename=package://sobit_pro/sobit_pro_description/meshes/sensor/mic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 scale=0.001 0.001 0.001
- link plate_bottom_link: geometry collision box size=0.3 0.3 0.009; visual mesh filename=package://sobit_pro/sobit_pro_description/meshes/body/plate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 scale=0.001 0.001 0.001
- link plate_middle_link: geometry collision box size=0.3 0.3 0.009; visual mesh filename=package://sobit_pro/sobit_pro_description/meshes/body/plate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 scale=0.001 0.001 0.001
- link plate_top_link: geometry collision box size=0.3 0.3 0.009; visual mesh filename=package://sobit_pro/sobit_pro_description/meshes/body/plate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 scale=0.001 0.001 0.001
- link wheel_b_l_drive_link: geometry collision cylinder length=0.029 radius=0.072; visual mesh filename=package://sobit_pro/sobit_pro_description/meshes/wheel/whee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 scale=0.001 0.001 0.001
- link wheel_b_l_steer_base_link: geometry collision box size=0.05525 0.0285 0.084; visual mesh filename=package://sobit_pro/sobit_pro_description/meshes/wheel/whee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 scale=0.001 0.001 0.001
- link wheel_b_l_steer_link: geometry collision box size=0.0436 0.0495 0.1766; visual mesh filename=package://sobit_pro/sobit_pro_description/meshes/wheel/whee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 scale=0.001 0.001 0.001
- link wheel_b_r_drive_link: geometry collision cylinder length=0.029 radius=0.072; visual mesh filename=package://sobit_pro/sobit_pro_description/meshes/wheel/whee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 scale=0.001 0.001 0.001
- link wheel_b_r_steer_base_link: geometry collision box size=0.05525 0.0285 0.084; visual mesh filename=package://sobit_pro/sobit_pro_description/meshes/wheel/whee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 scale=0.001 0.001 0.001
- link wheel_b_r_steer_link: geometry collision box size=0.0436 0.0495 0.1766; visual mesh filename=package://sobit_pro/sobit_pro_description/meshes/wheel/whee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 scale=0.001 0.001 0.001
- link wheel_f_l_drive_link: geometry collision cylinder length=0.029 radius=0.072; visual mesh filename=package://sobit_pro/sobit_pro_description/meshes/wheel/whee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 scale=0.001 0.001 0.001
- link wheel_f_l_steer_base_link: geometry collision box size=0.05525 0.0285 0.084; visual mesh filename=package://sobit_pro/sobit_pro_description/meshes/wheel/whee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 scale=0.001 0.001 0.001
- link wheel_f_l_steer_link: geometry collision box size=0.0436 0.0495 0.1766; visual mesh filename=package://sobit_pro/sobit_pro_description/meshes/wheel/whee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 scale=0.001 0.001 0.001
- link wheel_f_r_drive_link: geometry collision cylinder length=0.029 radius=0.072; visual mesh filename=package://sobit_pro/sobit_pro_description/meshes/wheel/whee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 scale=0.001 0.001 0.001
- link wheel_f_r_steer_base_link: geometry collision box size=0.05525 0.0285 0.084; visual mesh filename=package://sobit_pro/sobit_pro_description/meshes/wheel/whee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 scale=0.001 0.001 0.001
- link wheel_f_r_steer_link: geometry collision box size=0.0436 0.0495 0.1766; visual mesh filename=package://sobit_pro/sobit_pro_description/meshes/wheel/whee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 scale=0.001 0.001 0.001
