Commit message: [UPD] add robot ns, and detection range

File: sobit_pro_sim_description/urdf/sensor/lidar.urdf.xacro (robot description, xacro)
@@ -2,5 +2,5 @@
 <robot name="sobit_pro"
        xmlns:xacro="http://ros.org/wiki/xacro">
-  <xacro:macro name="lidar" params="prefix parent">
+  <xacro:macro name="lidar" params="prefix parent robot_namespace">
     <joint name="${prefix}_base_joint" type="fixed">
       <parent link="${parent}" />
@@ -30,5 +30,5 @@
       </inertial>
     </link>
-    <xacro:hokuyo_ust_mount prefix="${prefix}" parent="${prefix}_base_link" topic="scan" model="ust-10" >
+    <xacro:hokuyo_ust_mount prefix="${prefix}" parent="${prefix}_base_link" topic="scan" robot_namespace="${robot_namespace}/" model="ust-10" min_angle="-${M_PI/2}" max_angle="${M_PI/2}" >
       <origin xyz="0.067 0.0 0.0" rpy="0.0 0.0 0.0" />
     </xacro:hokuyo_ust_mount>

Commit message: [UPD] Isaac comment

File: sobit_pro_sim_description/urdf/sensor/lidar.urdf.xacro (robot description, xacro)
@@ -31,5 +31,8 @@
     </link>
     <xacro:hokuyo_ust_mount prefix="${prefix}" parent="${prefix}_base_link" topic="scan" robot_namespace="${robot_namespace}/" model="ust-10" min_angle="-${M_PI/2}" max_angle="${M_PI/2}" >
+      <!-- GZ -->
       <origin xyz="0.067 0.0 0.0" rpy="0.0 0.0 0.0" />
+      <!-- Isaac -->
+      <!-- <origin xyz="0.067 0.0 0.0" rpy="0.0 0.0 -${M_PI/2}" /> -->
     </xacro:hokuyo_ust_mount>
   </xacro:macro>

Commit message: [UPD] rotate 90 deg

File: sobit_pro_sim_description/urdf/sensor/lidar.urdf.xacro (robot description, xacro)
@@ -32,7 +32,7 @@
     <xacro:hokuyo_ust_mount prefix="${prefix}" parent="${prefix}_base_link" topic="scan" robot_namespace="${robot_namespace}/" model="ust-10" min_angle="-${M_PI/2}" max_angle="${M_PI/2}" >
       <!-- GZ -->
-      <origin xyz="0.067 0.0 0.0" rpy="0.0 0.0 0.0" />
+      <!-- <origin xyz="0.067 0.0 0.0" rpy="0.0 0.0 0.0" /> -->
       <!-- Isaac -->
-      <!-- <origin xyz="0.067 0.0 0.0" rpy="0.0 0.0 -${M_PI/2}" /> -->
+      <origin xyz="0.067 0.0 0.0" rpy="0.0 0.0 -${M_PI/2}" />
     </xacro:hokuyo_ust_mount>
   </xacro:macro>
